File: t-dsp_core.kicad_sch (KiCad schematic)
At the start: 163 parts, among them IC1 Logic Level Shifter - 74HCT2G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, J1 J_PWR, J10 J_DMX, J11 J_LED, J12 J_ETH, J2 J_TDM, J3 J_T, J4 J_USBH, J5 J_MIDI, J6 J_SPDIF, J7 J_AUX, J8 J_S3, J9 J_USB3, T108 Tab, T109 Tab, T110 Tab, T111 Tab, U1 Teensy 4.1 - DEVKIT, U11 Dual Buffer - SN74LVC2G125DCTR, U13 ESP32-S3-WROOM-1-N16R8, U15 LT3045EMSE#TRPBF, U16 THVD1450DR, U17 ISO7762DW, U18 TEA1-0505HI, U19 SRC4382IPFBR, U20 TLV75718PDRVR, U21 74LVC157APW, U22 IDC777-1, U23 74LVC157APW, U24 AP63203WU, U3 Power Mux & Protect - TPS2116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, U4 Optoisolators - H11L1SM - 6-S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, U5 Dual Buffer - SN74LVC2G125DCTR, U6 Dual Buffer - SN74LVC2G125DCTR, U7 Dual Buffer - SN74LVC2G125DCTR, U8 Dual Buffer - SN74LVC2G125DCTR, U9 Dual Buffer - 74HCT2G17GW,125, Y1 24.576MHz

Commit message: Spin 2 stage 10c: external-antenna build option; J13 u.FL (DNP) on IDC777/IDC767 pad 57 EXT_RF; antenna decision in change map
Co-Authored-By: Claude Fable 5.1 <noreply@anthropic.com>
Parts:
- added J13: u.FL DNP (IDC767 ext-antenna build only), Connector_Coaxial:U.FL_Hirose_U.FL-R-SMT-1_Vertical, symbol Connector:Conn_Coaxial
Connections:
- net GND: now also J13.2 (Ext)
- net BT_EXT_RF: now reaches U22.57 (EXT_RF)
- net BT_EXT_RF: now also J13.1 (In)
Other:
- note added: "J13 u.FL: DNP with the IDC777-1 (chip antenna). Fit J13 and populate U22 as IDC767 (same 60-pad LGA, pad 57 = EXT_RF) for an external antenna.\nPCB: 50 ohm CPW from pad 57 to J13, GND pads 56/58 either side, ground vias every 1-2 mm, keep it short, no matching network (IDC767-DTS-V003 p.8)."
Changed lines of the file:
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@@
     (diameter 0)
 )
+  (junction
+    (at 118.11 264.16)
+    (diameter 0)
+)
+  (junction
+    (at 104.14 266.7)
+    (diameter 0)
+)
+  (junction
+    (at -247.65 822.96)
+    (diameter 0)
+)
+  (junction
+    (at -227.33 822.96)
+    (diameter 0)
+)
+  (junction
+    (at -210.82 822.96)
+    (diameter 0)
+)
+  (junction
+    (at 118.11 264.16)
+    (diameter 0)
+)
+  (junction
+    (at 104.14 266.7)
+    (diameter 0)
+)
+  (junction
+    (at -247.65 822.96)
+    (diameter 0)
+)
+  (junction
+    (at -227.33 822.96)
+    (diameter 0)
+)
+  (junction
+    (at -210.82 822.96)
+    (diameter 0)
+)
+  (junction
+    (at 118.11 264.16)
+    (diameter 0)
+)
+  (junction
+    (at 104.14 266.7)
+    (diameter 0)
+)
+  (junction
+    (at -247.65 822.96)
+    (diameter 0)
+)
+  (junction
+    (at -227.33 822.96)
+    (diameter 0)
+)
+  (junction
+    (at -210.82 822.96)
+    (diameter 0)
+)
   (no_connect
     (at -229.87 916.94)
@@
       (xy 549.91 314.96))
 )
+  (wire
+    (pts
+      (xy 1330.96 582.93)
+      (xy 1328.42 582.93))
+)
+  (wire
+    (pts
+      (xy 1290.32 603.25)
+      (xy 1287.78 603.25))
+)
+  (wire
+    (pts
+      (xy 1295.4 608.33)
+      (xy 1295.4 610.87))
+)
   (text "https://electronics.stackexchange.com/questions/310899/midi-out-thru-circuit-questions"
     (at 819.15 852.17 0)
@@
       (justify left))
 )
+  (global_label "BT_EXT_RF"
+    (shape bidirectional)
+    (at 1328.42 582.93 180)
+    (effects
+      (font
+        (size 1.27 1.27))
+      (justify right))
+)
+  (global_label "BT_EXT_RF"
+    (shape bidirectional)
+    (at 1287.78 603.25 180)
+    (effects
+      (font
+        (size 1.27 1.27))
+      (justify right))
+)
+  (global_label "GND"
+    (shape bidirectional)
+    (at 1295.4 610.87 270)
+    (effects
+      (font
+        (size 1.27 1.27))
+      (justify right))
+)
   (symbol
     (lib_id "Device:R")
@@
           (reference "H4")
           (unit 1)))))
+  (symbol
+    (lib_id "Connector:Conn_Coaxial")
+    (at 1295.4 603.25 0)
+    (unit 1)
+    (in_bom yes)
+    (on_board yes)
+    (dnp no)
+    (property "Reference" "J13"
+      (at 1295.4 599.44 0)
+      (effects
+        (font
+          (size 1.27 1.27))))
+    (property "Value" "u.FL DNP (IDC767 ext-antenna build only)"
+      (at 1295.4 607.06 0)
+      (effects
+        (font
+          (size 1.27 1.27))))
+    (property "Footprint" "Connector_Coaxial:U.FL_Hirose_U.FL-R-SMT-1_Vertical"
+      (at 1295.4 603.25 0)
+      (effects
+        (font
+          (size 1.27 1.27))
+        (hide yes)))
+    (property "Datasheet" ""
+      (at 1295.4 603.25 0)
+      (effects
+        (font
+          (size 1.27 1.27))
+        (hide yes)))
+    (instances
+      (project "t-dsp_core"
+        (path "/6a0ff39d-771d-410f-9e7c-006586d81d16"
+          (reference "J13")
+          (unit 1)))))
   (rectangle
     (start 1008.38 845.82)
@@
     (path "/"
       (page "1")))
-)
+  (text "J13 u.FL: DNP with the IDC777-1 (chip antenna). Fit J13 and populate U22 as IDC767 (same 60-pad LGA, pad 57 = EXT_RF) for an external antenna.\\nPCB: 50 ohm CPW from pad 57 to J13, GND pads 56/58 either side, ground vias every 1-2 mm, keep it short, no matching network (IDC767-DTS-V003 p.8)."
+    (at 1280.16 618.49 0)
+    (effects (font (size 1.27 1.27)))
+  ))

Commit message: Spin 2 stage 10d: encoder nets become Teensy GPIO T_38/T_39/T_40 (A14-A16) on J8; S3 IO15/IO38/IO39 NC; backplane controls note and GPIO budget
Co-Authored-By: Claude Fable 5.1 <noreply@anthropic.com>
Connections:
- net OUTPUTA renamed T_40
- net T_40: no longer U13.31 (IO38)
- net OUTPUTB renamed T_39
- net T_39: no longer U13.32 (IO39)
- net SWITCH renamed T_38
- net T_38: no longer U13.8 (IO15)
- no-connect marks 60 -> 63
Other:
- note added: "Simple backplane controls (no extra parts on the core):\n Pot / volume knob: 10k linear between 3.3V (J1.9) and GND, wiper -> any T_ analog pin (T_22=A8, T_26=A12, T_27=A13, T_38=A14, T_39=A15, T_40=A16,\n T_BUTTON1=A10, T_BUTTON2=A11, 14_SPDIF_OUT=A0, 15_SPDIF_IN=A1) with 100 nF wiper-to-GND. analogRead(), average 8-16 samples.\n Switch / button: between a T_ pin and GND, pinMode(INPUT_PULLUP). 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"
Changed lines of the file:
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@@
     (at -240.03 631.19)
 )
+  (no_connect
+    (at -270.51 651.51)
+)
+  (no_connect
+    (at -240.03 633.73)
+)
+  (no_connect
+    (at -240.03 636.27)
+)
   (wire
     (pts
@@
   (wire
     (pts
-      (xy -270.51 651.51)
-      (xy -275.59 651.51))
-    (stroke
-      (width 0)
-      (type default))
-)
-  (wire
-    (pts
       (xy 287.02 227.33)
       (xy 295.91 227.33))
@@
   (wire
     (pts
-      (xy -240.03 633.73)
-      (xy -234.95 633.73))
-    (stroke
-      (width 0)
-      (type default))
-)
-  (wire
-    (pts
       (xy 1070.61 1120.14)
       (xy 1087.12 1120.14))
@@
   (wire
     (pts
-      (xy -240.03 636.27)
-      (xy -234.95 636.27))
-    (stroke
-      (width 0)
-      (type default))
-)
-  (wire
-    (pts
       (xy 1054.1 313.69)
       (xy 1062.99 313.69))
@@
         (size 1.27 1.27)))
 )
+  (text "J13 u.FL: DNP with the IDC777-1 (chip antenna). Fit J13 and populate U22 as IDC767 (same 60-pad LGA, pad 57 = EXT_RF) for an external antenna.\\nPCB: 50 ohm CPW from pad 57 to J13, GND pads 56/58 either side, ground vias every 1-2 mm, keep it short, no matching network (IDC767-DTS-V003 p.8)."
+    (at 1280.16 618.49 0)
+    (effects
+      (font
+        (size 1.27 1.27)))
+)
   (label "DMX_RO_ISO"
     (at -224.79 924.56 0)
@@
         (font
           (size 1.27 1.27)))))
-  (global_label "SWITCH"
-    (shape input)
-    (at -275.59 651.51 180)
-    (effects
-      (font
-        (size 1.27 1.27))
-      (justify right))
-    (property "Intersheetrefs" "${INTERSHEET_REFS}"
-      (at -275.59 651.51 0)
-      (hide yes)
-      (show_name no)
-      (do_not_autoplace no)
-      (effects
-        (font
-          (size 1.27 1.27)))))
   (global_label "GND"
     (shape input)
@@
           (size 1.27 1.27))
         (justify right))))
-  (global_label "OUTPUTA"
-    (shape input)
-    (at -234.95 633.73 0)
-    (effects
-      (font
-        (size 1.27 1.27))
-      (justify left))
-    (property "Intersheetrefs" "${INTERSHEET_REFS}"
-      (at -234.95 633.73 0)
-      (hide yes)
-      (show_name no)
-      (do_not_autoplace no)
-      (effects
-        (font
-          (size 1.27 1.27)))))
   (global_label "GND"
     (shape input)
@@
         (font
           (size 1.27 1.27)))))
-  (global_label "OUTPUTB"
-    (shape input)
-    (at -234.95 636.27 0)
-    (effects
-      (font
-        (size 1.27 1.27))
-      (justify left))
-    (property "Intersheetrefs" "${INTERSHEET_REFS}"
-      (at -234.95 636.27 0)
-      (hide yes)
-      (show_name no)
-      (do_not_autoplace no)
-      (effects
-        (font
-          (size 1.27 1.27)))))
   (global_label "GND"
     (shape input)
@@
       (justify right))
 )
-  (global_label "SWITCH"
-    (shape bidirectional)
-    (at 203.2 256.54 180)
-    (effects
-      (font
-        (size 1.27 1.27))
-      (justify right))
-)
-  (global_label "OUTPUTB"
-    (shape bidirectional)
-    (at 203.2 254 180)
-    (effects
-      (font
-        (size 1.27 1.27))
-      (justify right))
-)
-  (global_label "OUTPUTA"
-    (shape bidirectional)
-    (at 203.2 251.46 180)
-    (effects
-      (font
-        (size 1.27 1.27))
-      (justify right))
-)
   (global_label "ESP32_IO33_SPI_CS"
     (shape bidirectional)
@@
       (justify right))
 )
-  (global_label "OUTPUTA"
-    (shape bidirectional)
-    (at -90.17 624.84 0)
-    (effects
-      (font
-        (size 1.27 1.27))
-      (justify left))
-)
-  (global_label "OUTPUTB"
-    (shape bidirectional)
-    (at -107.95 627.38 180)
-    (effects
-      (font
-        (size 1.27 1.27))
-      (justify right))
-)
-  (global_label "SWITCH"
-    (shape bidirectional)
-    (at -90.17 627.38 0)
-    (effects
-      (font
-        (size 1.27 1.27))
-      (justify left))
-)
   (global_label "GND"
     (shape bidirectional)
@@
       (justify right))
 )
+  (global_label "T_38"
+    (shape bidirectional)
+    (at 203.2 256.54 180)
+    (effects
+      (font
+        (size 1.27 1.27))
+      (justify right))
+)
+  (global_label "T_39"
+    (shape bidirectional)
+    (at 203.2 254 180)
+    (effects
+      (font
+        (size 1.27 1.27))
+      (justify right))
+)
+  (global_label "T_40"
+    (shape bidirectional)
+    (at 203.2 251.46 180)
+    (effects
+      (font
+        (size 1.27 1.27))
+      (justify right))
+)
+  (global_label "T_40"
+    (shape bidirectional)
+    (at -90.17 624.84 0)
+    (effects
+      (font
+        (size 1.27 1.27))
+      (justify left))
+)
+  (global_label "T_39"
+    (shape bidirectional)
+    (at -107.95 627.38 180)
+    (effects
+      (font
+        (size 1.27 1.27))
+      (justify right))
+)
+  (global_label "T_38"
+    (shape bidirectional)
+    (at -90.17 627.38 0)
+    (effects
+      (font
+        (size 1.27 1.27))
+      (justify left))
+)
   (symbol
     (lib_id "Device:R")
@@
     (path "/"
       (page "1")))
-  (text "J13 u.FL: DNP with the IDC777-1 (chip antenna). Fit J13 and populate U22 as IDC767 (same 60-pad LGA, pad 57 = EXT_RF) for an external antenna.\\nPCB: 50 ohm CPW from pad 57 to J13, GND pads 56/58 either side, ground vias every 1-2 mm, keep it short, no matching network (IDC767-DTS-V003 p.8)."
-    (at 1280.16 618.49 0)
+  (text "Simple backplane controls (no extra parts on the core):\\n  Pot / volume knob: 10k linear between 3.3V (J1.9) and GND, wiper -> any T_ analog pin (T_22=A8, T_26=A12, T_27=A13, T_38=A14, T_39=A15, T_40=A16,\\n  T_BUTTON1=A10, T_BUTTON2=A11, 14_SPDIF_OUT=A0, 15_SPDIF_IN=A1) with 100 nF wiper-to-GND. analogRead(), average 8-16 samples.\\n  Switch / button: between a T_ pin and GND, pinMode(INPUT_PULLUP). More controls: 74HC4067 muxes on the analog pins,\\n  MCP23017 / TCA8418 on SDA1/SCL1 (J2), SK6812 chain on J11 for LEDs. T_38/T_39/T_40 are Teensy pins 38/39/40 on J8 pins 22/21/20."
+    (at -120.65 648.97 0)
     (effects (font (size 1.27 1.27)))
   ))

Commit message: Spin 2 stage 10e: S3 IO15/IO38/IO39 back on J8 as their own nets (pins 23/24/28); Teensy 38/39/40 and S3 pins now separate
Co-Authored-By: Claude Fable 5.1 <noreply@anthropic.com>
Connections:
- net GND: no longer J8.23 (Pin_23), J8.24 (Pin_24), J8.28 (Pin_28)
- net S3_IO38: now reaches U13.31 (IO38)
- net S3_IO38: now also J8.24 (Pin_24)
- net S3_IO39: now reaches U13.32 (IO39)
- net S3_IO39: now also J8.28 (Pin_28)
- net S3_IO15: now reaches U13.8 (IO15)
- net S3_IO15: now also J8.23 (Pin_23)
Changed lines of the file:
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@@
     (diameter 0)
 )
+  (junction
+    (at 118.11 264.16)
+    (diameter 0)
+)
+  (junction
+    (at 104.14 266.7)
+    (diameter 0)
+)
+  (junction
+    (at -247.65 822.96)
+    (diameter 0)
+)
+  (junction
+    (at -227.33 822.96)
+    (diameter 0)
+)
+  (junction
+    (at -210.82 822.96)
+    (diameter 0)
+)
+  (junction
+    (at 118.11 264.16)
+    (diameter 0)
+)
+  (junction
+    (at 104.14 266.7)
+    (diameter 0)
+)
+  (junction
+    (at -247.65 822.96)
+    (diameter 0)
+)
+  (junction
+    (at -227.33 822.96)
+    (diameter 0)
+)
+  (junction
+    (at -210.82 822.96)
+    (diameter 0)
+)
+  (junction
+    (at 118.11 264.16)
+    (diameter 0)
+)
+  (junction
+    (at 104.14 266.7)
+    (diameter 0)
+)
+  (junction
+    (at -247.65 822.96)
+    (diameter 0)
+)
+  (junction
+    (at -227.33 822.96)
+    (diameter 0)
+)
+  (junction
+    (at -210.82 822.96)
+    (diameter 0)
+)
   (no_connect
     (at -229.87 916.94)
@@
       (xy 1295.4 610.87))
 )
+  (wire
+    (pts
+      (xy -270.51 651.51)
+      (xy -275.59 651.51))
+)
+  (wire
+    (pts
+      (xy -240.03 633.73)
+      (xy -234.95 633.73))
+)
+  (wire
+    (pts
+      (xy -240.03 636.27)
+      (xy -234.95 636.27))
+)
   (text "https://electronics.stackexchange.com/questions/310899/midi-out-thru-circuit-questions"
     (at 819.15 852.17 0)
@@
         (size 1.27 1.27)))
 )
+  (text "Simple backplane controls (no extra parts on the core):\\n  Pot / volume knob: 10k linear between 3.3V (J1.9) and GND, wiper -> any T_ analog pin (T_22=A8, T_26=A12, T_27=A13, T_38=A14, T_39=A15, T_40=A16,\\n  T_BUTTON1=A10, T_BUTTON2=A11, 14_SPDIF_OUT=A0, 15_SPDIF_IN=A1) with 100 nF wiper-to-GND. analogRead(), average 8-16 samples.\\n  Switch / button: between a T_ pin and GND, pinMode(INPUT_PULLUP). More controls: 74HC4067 muxes on the analog pins,\\n  MCP23017 / TCA8418 on SDA1/SCL1 (J2), SK6812 chain on J11 for LEDs. T_38/T_39/T_40 are Teensy pins 38/39/40 on J8 pins 22/21/20."
+    (at -120.65 648.97 0)
+    (effects
+      (font
+        (size 1.27 1.27)))
+)
   (label "DMX_RO_ISO"
     (at -224.79 924.56 0)
@@
       (justify right))
 )
-  (global_label "GND"
-    (shape bidirectional)
-    (at -107.95 629.92 180)
-    (effects
-      (font
-        (size 1.27 1.27))
-      (justify right))
-)
-  (global_label "GND"
-    (shape bidirectional)
-    (at -90.17 629.92 0)
-    (effects
-      (font
-        (size 1.27 1.27))
-      (justify left))
-)
   (global_label "GPIO34"
     (shape bidirectional)
@@
       (justify right))
 )
-  (global_label "GND"
-    (shape bidirectional)
-    (at -90.17 635 0)
-    (effects
-      (font
-        (size 1.27 1.27))
-      (justify left))
-)
   (global_label "ETH_R+"
     (shape bidirectional)
@@
       (justify left))
 )
+  (global_label "S3_IO15"
+    (shape bidirectional)
+    (at -275.59 651.51 180)
+    (effects
+      (font
+        (size 1.27 1.27))
+      (justify right))
+)
+  (global_label "S3_IO38"
+    (shape bidirectional)
+    (at -234.95 633.73 0)
+    (effects
+      (font
+        (size 1.27 1.27))
+      (justify left))
+)
+  (global_label "S3_IO39"
+    (shape bidirectional)
+    (at -234.95 636.27 0)
+    (effects
+      (font
+        (size 1.27 1.27))
+      (justify left))
+)
+  (global_label "S3_IO15"
+    (shape bidirectional)
+    (at -107.95 629.92 180)
+    (effects
+      (font
+        (size 1.27 1.27))
+      (justify right))
+)
+  (global_label "S3_IO38"
+    (shape bidirectional)
+    (at -90.17 629.92 0)
+    (effects
+      (font
+        (size 1.27 1.27))
+      (justify left))
+)
+  (global_label "S3_IO39"
+    (shape bidirectional)
+    (at -90.17 635 0)
+    (effects
+      (font
+        (size 1.27 1.27))
+      (justify left))
+)
   (symbol
     (lib_id "Device:R")
@@
     (path "/"
       (page "1")))
-  (text "Simple backplane controls (no extra parts on the core):\\n  Pot / volume knob: 10k linear between 3.3V (J1.9) and GND, wiper -> any T_ analog pin (T_22=A8, T_26=A12, T_27=A13, T_38=A14, T_39=A15, T_40=A16,\\n  T_BUTTON1=A10, T_BUTTON2=A11, 14_SPDIF_OUT=A0, 15_SPDIF_IN=A1) with 100 nF wiper-to-GND. analogRead(), average 8-16 samples.\\n  Switch / button: between a T_ pin and GND, pinMode(INPUT_PULLUP). More controls: 74HC4067 muxes on the analog pins,\\n  MCP23017 / TCA8418 on SDA1/SCL1 (J2), SK6812 chain on J11 for LEDs. T_38/T_39/T_40 are Teensy pins 38/39/40 on J8 pins 22/21/20."
-    (at -120.65 648.97 0)
-    (effects (font (size 1.27 1.27)))
-  ))
+)

Commit message: Spin 2 stage 10f: header GPIO net-naming rule; 42 nets renamed to T<pin> / S3_IO<gpio> (fixes three wrong S3 GPIO numbers); topology unchanged
Co-Authored-By: Claude Fable 5.1 <noreply@anthropic.com>
Connections:
- net 14_SPDIF_OUT renamed T14_SPDIF_OUT
- net 15_SPDIF_IN renamed T15_SPDIF_IN
- net 32_OUT1B renamed T32_OUT1B
- net 34_RX8_RESET2 renamed T34_RX8
- net 35_TX8_RESET renamed T35_TX8
- net 53_T_PROG renamed T_PROGRAM
- net 54_ON_OFF renamed T_ON_OFF
- net CRX3 renamed T30_CRX3
- net CS renamed S3_IO11
- net DC renamed S3_IO2
- net ESP32_EN renamed S3_EN
- net ESP32_IO0 renamed S3_IO0_BOOT
- net ESP32_IO1 renamed S3_IO43_TXD0
- net ESP32_IO12_SPI_MISO renamed S3_IO12_SPI_MISO
- net ESP32_IO13_SPI_MOSI renamed S3_IO13_SPI_MOSI
- net ESP32_IO14_SPI_SCK renamed S3_IO14_SPI_SCK
- net ESP32_IO21_SDA renamed S3_IO21_SDA
- net ESP32_IO22_SCL renamed S3_IO47_SCL
- net ESP32_IO3 renamed S3_IO44_RXD0
- net ESP32_IO33_SPI_CS renamed S3_IO17_SPI_CS
- net ESP32_LED renamed S3_IO46_LED
- net GPIO34 renamed S3_IO40
- net GPIO35 renamed S3_IO41
- net MCLK2 renamed T33_MCLK2
- net RESET renamed S3_IO42
- net SCK renamed S3_IO18
- net SCL0 renamed T19_SCL0
- net SCL1 renamed T16_SCL1
- net SDA0 renamed T18_SDA0
- net SDA1 renamed T17_SDA1
- net SDI renamed S3_IO9
- net SDO renamed S3_IO10
- net TRX3 renamed T31_CTX3
- net T_22 renamed T22
- net T_26 renamed T26
- net T_27 renamed T27
- net T_38 renamed T38
- net T_39 renamed T39
- net T_40 renamed T40
- net T_BUTTON1 renamed T24
- net T_BUTTON2 renamed T25
- net T_CS renamed S3_IO8
Other:
- note added: "Header net naming: functions keep function names (TDM, SPDIF, USB, MIDI, DMX, LED, power); raw GPIO is named by MCU pin: T<n> = Teensy 4.1 pin n,\nS3_IO<n> = ESP32-S3 GPIO n; an optional core function rides as a suffix (T14_SPDIF_OUT, T35_TX8, T18_SDA0, S3_IO43_TXD0, S3_IO47_SCL).\nSimple backplane controls (no extra parts on the core): pot / volume knob = 10k linear between 3.3V (J1.9) and GND, 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"
- note removed: "Simple backplane controls (no extra parts on the core):\n Pot / volume knob: 10k linear between 3.3V (J1.9) and GND, wiper -> any T_ analog pin (T_22=A8, T_26=A12, T_27=A13, T_38=A14, T_39=A15, T_40=A16,\n T_BUTTON1=A10, T_BUTTON2=A11, 14_SPDIF_OUT=A0, 15_SPDIF_IN=A1) with 100 nF wiper-to-GND. analogRead(), average 8-16 samples.\n Switch / button: between a T_ pin and GND, pinMode(INPUT_PULLUP). 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"
