File: t-dsp_core.kicad_sch (KiCad schematic)
At the start: 164 parts, among them IC1 Logic Level Shifter - 74HCT2G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, J1 J_PWR, J10 J_DMX, J11 J_LED, J12 J_ETH, J13 u.FL DNP (IDC767 ext-antenna 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, J2 J_TDM, J3 J_T, J4 J_USBH, J5 J_MIDI, J6 J_SPDIF, J7 J_AUX, J8 J_S3, J9 J_USB3, T108 Tab, T109 Tab, T110 Tab, T111 Tab, U1 Teensy 4.1 - DEVKIT, U11 Dual Buffer - SN74LVC2G125DCTR, U13 ESP32-S3-WROOM-1-N16R8, U15 LT3045EMSE#TRPBF, U16 THVD1450DR, U17 ISO7762DW, U18 TEA1-0505HI, U19 SRC4382IPFBR, U20 TLV75718PDRVR, U21 74LVC157APW, U22 IDC777-1, U23 74LVC157APW, U24 AP63203WU, U3 Power Mux & Protect - TPS2116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, U4 Optoisolators - H11L1SM - 6-S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, U5 Dual Buffer - SN74LVC2G125DCTR, U6 Dual Buffer - SN74LVC2G125DCTR, U7 Dual Buffer - SN74LVC2G125DCTR, U8 Dual Buffer - SN74LVC2G125DCTR, U9 Dual Buffer - 74HCT2G17GW,125, Y1 24.576MHz

Commit message: Spin 2 stage 10g: MIDI passives out of the ESP32 antenna keep-out, 3.3V caps to the left column, holes at the corners, plain 3.2 mm hole footprint; schematic restored after a stale eeschema save
Co-Authored-By: Claude Fable 5.1 <noreply@anthropic.com>
Parts:
- H1, H2, H3, H4: footprint MountingHole:MountingHole_3.2mm_M3 -> MountingHole:MountingHole_3.2mm
Changed lines of the file:
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@@
         (font
           (size 1.27 1.27))))
-    (property "Footprint" "MountingHole:MountingHole_3.2mm_M3"
+    (property "Footprint" "MountingHole:MountingHole_3.2mm"
       (at 1029.97 640.08 0)
       (effects
@@
         (font
           (size 1.27 1.27))))
-    (property "Footprint" "MountingHole:MountingHole_3.2mm_M3"
+    (property "Footprint" "MountingHole:MountingHole_3.2mm"
       (at 1060.45 640.08 0)
       (effects
@@
         (font
           (size 1.27 1.27))))
-    (property "Footprint" "MountingHole:MountingHole_3.2mm_M3"
+    (property "Footprint" "MountingHole:MountingHole_3.2mm"
       (at 1090.93 640.08 0)
       (effects
@@
         (font
           (size 1.27 1.27))))
-    (property "Footprint" "MountingHole:MountingHole_3.2mm_M3"
+    (property "Footprint" "MountingHole:MountingHole_3.2mm"
       (at 1121.41 640.08 0)
       (effects

Commit message: D3/D4 to SK6812-EC20: value, project_fp:LED_SK6812-EC20_2.0x2.0mm footprint, LCSC C2909058 (schematic file re-saved by eeschema, netlist unchanged)
Co-Authored-By: Claude Fable 5.1 <noreply@anthropic.com>
Parts:
- D3, D4: value Side Light LED - SK6812 -> SK6812-EC20; footprint project_fp:SK6812-32228SMD-Reverse-Mount_mod -> project_fp:LED_SK6812-EC20_2.0x2.0mm; LCSC C5378721 -> C2909058; LCSC_MPN SK6812SIDE-A -> SK6812-EC20

Commit message: Spin 2 stage 10m: J9 folded into J8 (2x17: S3 USB pair + 5V, GND flanked), J1 trimmed to 2x5, H1-H4 back on MountingHole_3.2mm_M3, stale NC flags on S3 IO15/38/39 and IDC777 EXT_RF removed
Co-Authored-By: Claude Fable 5.1 <noreply@anthropic.com>
Parts:
- removed J9: J_USB3, Connector_PinHeader_2.54mm:PinHeader_1x05_P2.54mm_Vertical, symbol Connector_Generic:Conn_01x05
- H1, H2, H3, H4: footprint MountingHole:MountingHole_3.2mm -> MountingHole:MountingHole_3.2mm_M3
- J1: footprint Connector_PinHeader_2.54mm:PinHeader_2x06_P2.54mm_Vertical -> Connector_PinHeader_2.54mm:PinHeader_2x05_P2.54mm_Vertical; symbol Connector_Generic:Conn_02x06_Odd_Even -> Connector_Generic:Conn_02x05_Odd_Even
- J8: footprint Connector_PinHeader_2.54mm:PinHeader_2x15_P2.54mm_Vertical -> Connector_PinHeader_2.54mm:PinHeader_2x17_P2.54mm_Vertical; symbol Connector_Generic:Conn_02x15_Odd_Even -> Connector_Generic:Conn_02x17_Odd_Even
Connections:
- net 3.3V: now also J1.7 (Pin_7); no longer J1.9 (Pin_9)
- net 3.3V_DIG: now also J1.8 (Pin_8); no longer J1.10 (Pin_10)
- net 5V: now also J8.34 (Pin_34)
- net GND: now also J1.10 (Pin_10), J8.33 (Pin_33); no longer J1.12 (Pin_12), J1.7 (Pin_7), J1.8 (Pin_8)
- net S3_USB_DN: now also J8.31 (Pin_31)
- net S3_USB_DP: now also J8.32 (Pin_32)
- net V_BAT: now also J1.9 (Pin_9); no longer J1.11 (Pin_11)
- no-connect marks 63 -> 59

Commit message: Spin 2 stage 10n: outer header rows at the board edges between the corner holes (J3/J12 left, J8 right; J4 to row B, J1 to row C, J10/J11 into slot 2); 0805 passives to 0603 JLC basic parts (51 caps, 52 resistors, LCSC fields updated, 2.21k -> 2.2k); board footprints/values/fields synced via pcbnew; passives re-placed two-sided
Passive-to-pin median 2.2 mm (was 9.9 at stage 10l), 6 of 118 > 10 mm. DRC: only the stock ESP32
courtyard overlaps and inherited drill warnings; schematic parity clean apart from the board_outline2
footprint that has never had a symbol.

Co-Authored-By: Claude Fable 5.1 <noreply@anthropic.com>
Parts:
- C1, C29, C30: footprint project_fp:C_0805_2012Metric_Pad1.15x1.40mm_HandSolder -> Capacitor_SMD:C_0603_1608Metric; LCSC C6119929 -> C15849; LCSC_MPN CGA0805X7R105K500MT -> CL10A105KB8NNNC
- C12, C13, C23, C31, C33, C34, C44: footprint project_fp:C_0805_2012Metric_Pad1.15x1.40mm_HandSolder -> Capacitor_SMD:C_0603_1608Metric; LCSC C15850 -> C19702; LCSC_MPN CL21A106KAYNNNE -> CL10A106KP8NNNC
- C130, C135, C138, C139, C144, C145, C148, C151: footprint project_fp:C_0805_2012Metric_Pad1.15x1.40mm_HandSolder -> Capacitor_SMD:C_0603_1608Metric; LCSC C15850 -> C19702
- C131, C133, C134, C136, C137, C140, C141, C142, C143, C146, C149, C150, C152, C153, C4, C5: footprint project_fp:C_0805_2012Metric_Pad1.15x1.40mm_HandSolder -> Capacitor_SMD:C_0603_1608Metric; LCSC C49678 -> C14663
- C14, C16, C17, C18, C19, C2, C20, C21, C22, C3, C32, C35, C40: footprint project_fp:C_0805_2012Metric_Pad1.15x1.40mm_HandSolder -> Capacitor_SMD:C_0603_1608Metric; LCSC C49678 -> C14663; LCSC_MPN CC0805KRX7R9BB104 -> CC0603KRX7R9BB104
- C147: footprint project_fp:C_0805_2012Metric_Pad1.15x1.40mm_HandSolder -> Capacitor_SMD:C_0603_1608Metric; LCSC C6119929 -> C15849
- C41, C42: footprint project_fp:C_0805_2012Metric_Pad1.15x1.40mm_HandSolder -> Capacitor_SMD:C_0603_1608Metric; LCSC C15850 -> C19702; LCSC_MPN (none) -> CL10A106KP8NNNC
- C43: footprint project_fp:C_0805_2012Metric_Pad1.15x1.40mm_HandSolder -> Capacitor_SMD:C_0603_1608Metric; LCSC C1779 -> C19666; LCSC_MPN (none) -> CL10A475KO8NNNC
- R1, R10, R2, R3, R4, R40, R41, R42, R43, R44, R45, R46, R47, R5, R52, R55, R56, R6, R7, R9: footprint project_fp:R_0805_2012Metric_Pad1.15x1.40mm_HandSolder -> Resistor_SMD:R_0603_1608Metric; LCSC C17720 -> C23185; LCSC_MPN 0805W8F499JT5E -> 0603WAF499JT5E
- R11, R54: footprint project_fp:R_0805_2012Metric_Pad1.15x1.40mm_HandSolder -> Resistor_SMD:R_0603_1608Metric; LCSC C17414 -> C25804; LCSC_MPN 0805W8F1002T5E -> 0603WAF1002T5E
- R12, R15, R31, R35: footprint project_fp:R_0805_2012Metric_Pad1.15x1.40mm_HandSolder -> Resistor_SMD:R_0603_1608Metric; LCSC C17477 -> C21189; LCSC_MPN 0805W8F0000T5E -> 0603WAF0000T5E
- R13, R14, R16, R17, R67, R68: value 2.21k ohm -> 2.2k ohm; footprint project_fp:R_0805_2012Metric_Pad1.15x1.40mm_HandSolder -> Resistor_SMD:R_0603_1608Metric; LCSC C17520 -> C4190; LCSC_MPN 0805W8F2201T5E -> 0603WAF2201T5E
- R19, R53, R73: footprint project_fp:R_0805_2012Metric_Pad1.15x1.40mm_HandSolder -> Resistor_SMD:R_0603_1608Metric; LCSC C17414 -> C25804
- R29, R30: footprint project_fp:R_0805_2012Metric_Pad1.15x1.40mm_HandSolder -> Resistor_SMD:R_0603_1608Metric; LCSC C27834 -> C23186; LCSC_MPN 0805W8F5101T5E -> 0603WAF5101T5E
- R32, R34, R36, R37, R38, R39, R8: footprint project_fp:R_0805_2012Metric_Pad1.20x1.40mm_HandSolder -> Resistor_SMD:R_0603_1608Metric; LCSC C17557 -> C22962; LCSC_MPN 0805W8F2200T5E -> 0603WAF2200T5E
- R33: footprint project_fp:R_0805_2012Metric_Pad1.15x1.40mm_HandSolder -> Resistor_SMD:R_0603_1608Metric; LCSC C4310 -> C22843; LCSC_MPN 0805W8F1501T5E -> 0603WAF1501T5E
- R57: footprint project_fp:R_0805_2012Metric_Pad1.15x1.40mm_HandSolder -> Resistor_SMD:R_0603_1608Metric; LCSC C17633 -> C4216; LCSC_MPN (none) -> 0603WAF3302T5E
- R58: footprint project_fp:R_0805_2012Metric_Pad1.15x1.40mm_HandSolder -> Resistor_SMD:R_0603_1608Metric; LCSC C17617 -> C23025; LCSC_MPN (none) -> 0603WAF3000T5E
- R61: footprint project_fp:R_0805_2012Metric_Pad1.15x1.40mm_HandSolder -> Resistor_SMD:R_0603_1608Metric; LCSC C17634 -> C23140; LCSC_MPN (none) -> 0603WAF330JT5E
- R66, R72: footprint project_fp:R_0805_2012Metric_Pad1.15x1.40mm_HandSolder -> Resistor_SMD:R_0603_1608Metric; LCSC C17407 -> C25803
- R71: footprint project_fp:R_0805_2012Metric_Pad1.15x1.40mm_HandSolder -> Resistor_SMD:R_0603_1608Metric; LCSC C17437 -> C22787

Commit message: Spin 2 stage 10r: TDM fan-out buffers U5-U8 (4x SN74LVC2G125) replaced by one SN74LVC541APWR (U5, LCSC C113281); OE1 grounded (TDM1 group), OE2 = TDM2_OE via bridged solder jumper JP1 with 10k pull-up R74 so the TDM2 clock/data copies can be tri-stated for an external clock master; C18-C20 removed; U11 stays for the Teensy-input lines
Netlist verified: all other connectivity identical; new nets TDM1/TDM2_*_B between U5 and R40-R47, TDM2_OE.

Co-Authored-By: Claude Fable 5.1 <noreply@anthropic.com>
Parts:
- removed C18, C19, C20: 0.1 uF, Capacitor_SMD:C_0603_1608Metric, symbol Device:C_Small
- removed U5, U6, U7, U8: Dual Buffer - SN74LVC2G125DCTR, project_fp:SOP65P400X130-8N, symbol SN74LVC2G125DCTR:SN74LVC2G125DCTR
- added JP1: SJ bridged, Jumper:SolderJumper-2_P1.3mm_Bridged_Pad1.0x1.5mm, symbol Device:R
- added R74: 10k, Resistor_SMD:R_0603_1608Metric, symbol Device:R
- added U5: SN74LVC541APWR, Package_SO:TSSOP-20_4.4x6.5mm_P0.65mm, symbol 74xx:74LS541
Connections:
- net 3.3V: now also R74.1, U5.20 (VCC)
- net 6_OUT1D: now also U5.9 (A7)
- net 7_OUT1A: now also U5.5 (A3)
- net BCLK1: now also U5.4 (A2), U5.8 (A6)
- net GND: now also JP1.2, U5.1 (G1), U5.10 (GND)
- net LRCK1: now also U5.2 (A0), U5.6 (A4)
- net MCLK1: now also U5.3 (A1), U5.7 (A5)
- net TDM2_LRCK_B: now reaches R43.1
- net TDM2_LRCK_B: now also U5.14 (Y4)
- net TDM1_BCLK_B: now reaches R44.1
- net TDM1_BCLK_B: now also U5.16 (Y2)
- net TDM1_DOUT_B: now reaches R46.1
- net TDM1_DOUT_B: now also U5.15 (Y3)
- net TDM2_DOUT_B: now reaches R47.1
- net TDM2_DOUT_B: now also U5.11 (Y7)
- net TDM2_BCLK_B: now reaches R45.1
- net TDM2_BCLK_B: now also U5.12 (Y6)
- net TDM1_LRCK_B: now reaches R42.1
- net TDM1_LRCK_B: now also U5.18 (Y0)
- net TDM2_MCLK_B: now reaches R40.1
- net TDM2_MCLK_B: now also U5.13 (Y5)
- net TDM1_MCLK_B: now reaches R41.1
- net TDM1_MCLK_B: now also U5.17 (Y1)
- new net TDM2_OE: JP1.1, R74.2, U5.19 (G2)

Commit message: Spin 2 stage 10u: the 20 clock/data series terminations (R1-R7, R9, R10, R40-R47, R52, R55, R56) 49.9 ohm 0603 -> 33 ohm 0402 JLCPCB basic part (Uniroyal 0402WGF330JTCE, LCSC C25105); user accepted 22-100 ohm, easy sourcing
Co-Authored-By: Claude Fable 5.1 <noreply@anthropic.com>
Parts:
- R1, R10, R2, R3, R4, R40, R41, R42, R43, R44, R45, R46, R47, R5, R52, R55, R56, R6, R7, R9: value 49.9 ohm -> 33 ohm; footprint Resistor_SMD:R_0603_1608Metric -> Resistor_SMD:R_0402_1005Metric; LCSC C23185 -> C25105; LCSC_MPN 0603WAF499JT5E -> 0402WGF330JTCE

Commit message: Spin 2 stage 10v: switchable-direction buffers for Teensy OUT1B and OUT1C. U6 (2G125) buffers OUT1B both ways to the new J2 pin 27 (J2 now 2x14, pin 28 GND); U7 (2G125) adds the output direction for OUT1C alongside the existing U11 input half. Direction per line by 0 ohm jumper pairs: OUT1B out by default (R77/R80 fitted, R78/R79 DNP), OUT1C in by default (R83/R84 fitted, R82/R85 DNP). 33 ohm series R75/R76/R81, decoupling C18/C19.
Netlist verified: every other connection unchanged; ERC at the baseline.

Co-Authored-By: Claude Fable 5.1 <noreply@anthropic.com>
Parts:
- added C18, C19: 100nF, Capacitor_SMD:C_0603_1608Metric, symbol Device:C_Small
- added R75, R76, R81: 33 ohm, Resistor_SMD:R_0402_1005Metric, symbol Device:R
- added R77, R80, R83, R84: 0 ohm, Resistor_SMD:R_0402_1005Metric, symbol Device:R
- added R78, R79, R82, R85: 0 ohm DNP, Resistor_SMD:R_0402_1005Metric, symbol Device:R
- added U6, U7: SN74LVC2G125DCTR, project_fp:SOP65P400X130-8N, symbol SN74LVC2G125DCTR:SN74LVC2G125DCTR
- J2: footprint Connector_PinHeader_2.54mm:PinHeader_2x13_P2.54mm_Vertical -> Connector_PinHeader_2.54mm:PinHeader_2x14_P2.54mm_Vertical; symbol Connector_Generic:Conn_02x13_Odd_Even -> Connector_Generic:Conn_02x14_Odd_Even
Connections:
- net 3.3V: now also C18.1, C19.1, R78.2, R80.2, R83.2, R85.2, U6.8 (VCC), U7.7 (~{2OE}), U7.8 (VCC)
- net 9_OUT1C_INPUT: now also R81.2
- net 9_OUT1C_INPUT+: now also U7.2 (1A)
- net GND: now also J2.28 (Pin_28), C18.2, C19.2, R77.2, R79.2, R82.2, R84.2, U6.4 (GND), U7.4 (GND), U7.5 (2A); no longer U11.7 (~{2OE})
- net OUT1B_MCU: now reaches R5.2, U1.24 (32_OUT1B)
- net OUT1B_MCU: now also R76.2, U6.2 (1A)
- new net: R81.1, U7.6 (1Y)
- new net: R75.1, U6.6 (1Y)
- new net: R76.1, U6.3 (2Y)
- new net 32_OUT1B: J2.27 (Pin_27), R75.2, U6.5 (2A)
- new net OUT1B_OE_IN: R79.1, R80.1, U6.7 (~{2OE})
- new net OUT1B_OE_OUT: R77.1, R78.1, U6.1 (~{1OE})
- new net OUT1C_OE_IN: R84.1, R85.1, U11.7 (~{2OE})
- new net OUT1C_OE_OUT: R82.1, R83.1, U7.1 (~{1OE})
- no-connect marks 59 -> 60

Commit message: Spin 2 stage 10x (1/2): external supply mandatory. TPS2116 mux + PR1 divider + Teensy-USB caps removed, Teensy VUSB NC; 5V_IN -> SMAJ5.0A TVS (D7) -> AO3401A reverse-polarity P-FET (Q1) -> 5V rail with PWR_FLAG. USB isolation prep: J4 is a 2x5 J_USB (host row + Teensy device laptop-side row), Teensy pads 66/67 labelled, S3 USB nets split into laptop side (J8 31-34: DN, DP, S3_USB_GND, S3_VBUS) and module side; ISOUSB211DPR symbol + SSOP-28 footprint created, library registered
Netlist: all other connectivity identical; the new USB nets are single-node until the two
isolators are placed (manual eeschema step, change map 11.7).

Co-Authored-By: Claude Fable 5.1 <noreply@anthropic.com>
Parts:
- removed C13: 10 uF, Capacitor_SMD:C_0603_1608Metric, symbol TEENSY_4.0_ESP32_AUDIO-rescue:C_Small-Device
- removed C14: 0.1 uF, Capacitor_SMD:C_0603_1608Metric, symbol TEENSY_4.0_ESP32_AUDIO-rescue:C_Small-Device
- removed R28: 16.9k ohm, project_fp:R_0805_2012Metric_Pad1.15x1.40mm_HandSolder, symbol Device:R
- removed R29, R30: 5.1k ohm, Resistor_SMD:R_0603_1608Metric, symbol Device:R
- removed U3: Power Mux & Protect - TPS2116DRL, project_fp:TPS2116DRL, symbol Power_Management:TPS2116DRL
- added D7: SMAJ5.0A, Diode_SMD:D_SMA, symbol Device:D_Zener
- added Q1: AO3401A, Package_TO_SOT_SMD:SOT-23, symbol Transistor_FET:Q_PMOS_GSD
- J4: value J_USBH -> J_USB; footprint Connector_PinHeader_2.54mm:PinHeader_1x05_P2.54mm_Vertical -> Connector_PinHeader_2.54mm:PinHeader_2x05_P2.54mm_Vertical; symbol Connector_Generic:Conn_01x05 -> Connector_Generic:Conn_02x05_Odd_Even
Connections:
- net 5V: now also Q1.2 (S); no longer J8.34 (Pin_34)
- net 5V_IN: now also D7.1 (K), Q1.3 (D)
- net GND: now also J4.7 (Pin_7), D7.2 (A), Q1.1 (G); no longer J4.4 (Pin_4), J8.33 (Pin_33)
- net HOST_5V: now also J4.9 (Pin_9); no longer J4.5 (Pin_5)
- net HOST_D1+: now also J4.5 (Pin_5); no longer J4.3 (Pin_3)
- net HOST_D1-: now also J4.3 (Pin_3); no longer J4.2 (Pin_2)
- net S3_USB_DN: no longer U13.13 (USB_D-)
- net S3_USB_DP: no longer U13.14 (USB_D+)
- net T_USB_DN_M: now reaches U1.66 (D-)
- net T_USB_DP_M: now reaches U1.67 (D+)
- net 5V_VUSB: no longer names the net of U1.49 (VUSB)
- new net S3_USB_DN_M: U13.13 (USB_D-)
- new net S3_USB_DP_M: U13.14 (USB_D+)
- new net S3_USB_GND: J8.33 (Pin_33)
- new net S3_VBUS: J8.34 (Pin_34)
- new net T_USB_DN: J4.4 (Pin_4)
- new net T_USB_DP: J4.6 (Pin_6)
- new net T_USB_GND: J4.2 (Pin_2), J4.8 (Pin_8)
- new net T_VBUS: J4.10 (Pin_10)
- no-connect marks 60 -> 59
